Commit message: Added correct limits for urdf

File: install/eezybotarm_control/share/eezybotarm_control/description/eezybotarm.urdf.xacro (robot description, xacro)
@@ -34,5 +34,4 @@
         <axis xyz="0 0 1"/>
         <limit effort="100" velocity="1.0" lower="-0.7854" upper="0.7854"/>
-        <!-- [-45,45] degrees -->
     </joint>
     <!-- LINK 1 -->
@@ -58,5 +57,5 @@
         <child link="link_2"/>
         <axis xyz="0 0 1"/>
-        <limit effort="100" velocity="1.0" lower="-0.6109" upper="0.9599"/>
+        <limit effort="100" velocity="1.0" lower="-0.279253" upper="1.01229"/>
         <!-- [-35,55] degrees -->
     </joint>
@@ -83,5 +82,5 @@
         <child link="link_3"/>
         <axis xyz="0 0 1"/>
-        <limit effort="100" velocity="1.0" lower="-1.2217" upper="0.3491"/>
+        <limit effort="100" velocity="1.0" lower="0" upper="1.22173"/>
         <!-- [-70,20] degrees -->
     </joint>

Commit message: fixed urdf limits

File: install/eezybotarm_control/share/eezybotarm_control/description/eezybotarm.urdf.xacro (robot description, xacro)
@@ -27,11 +27,12 @@
         </collision>
     </link>
-    <!-- JOINT 1 -->
+    <!-- JOINT 1 (Base rotation) -->
     <joint name="joint_1" type="revolute">
         <origin xyz="0 0 0.05" rpy="0 0 0"/>
         <parent link="base_link"/>
         <child link="link_1"/>
-        <axis xyz="0 0 1"/>
+        <axis xyz="0 0 -1"/>
         <limit effort="100" velocity="1.0" lower="-0.7854" upper="0.7854"/>
+        <!-- [-45,45] degrees -->
     </joint>
     <!-- LINK 1 -->
@@ -51,10 +52,11 @@
         </collision>
     </link>
-    <!-- JOINT 2 -->
+    <!-- JOINT 2 (Shoulder) -->
     <joint name="joint_2" type="revolute">
         <origin xyz="0 -0.005 0.035" rpy="1.578 0 0"/>
         <parent link="link_1"/>
         <child link="link_2"/>
-        <axis xyz="0 0 1"/>
+        <axis xyz="0 0 -1"/>
+        <!-- <limit effort="100" velocity="1.0" lower="-1.01229" upper="0.279253"/> -->
         <limit effort="100" velocity="1.0" lower="-0.279253" upper="1.01229"/>
         <!-- [-35,55] degrees -->
@@ -76,10 +78,10 @@
         </collision>
     </link>
-    <!-- JOINT 3 -->
+    <!-- JOINT 3 (Elbow) -->
     <joint name="joint_3" type="revolute">
         <origin xyz="-0.021 0.133 -0.0105" rpy="0 0 0"/>
         <parent link="link_2"/>
         <child link="link_3"/>
-        <axis xyz="0 0 1"/>
+        <axis xyz="0 0 -1"/>
         <limit effort="100" velocity="1.0" lower="0" upper="1.22173"/>
         <!-- [-70,20] degrees -->
@@ -101,31 +103,3 @@
         </collision>
     </link>
-    <!-- Add transmission elements for ros2_control -->
-    <transmission name="joint_1_trans">
-        <type>transmission_interface/SimpleTransmission</type>
-        <joint name="joint_1">
-            <hardwareInterface>hardware_interface/PositionJointInterface</hardwareInterface>
-        </joint>
-        <actuator name="joint_1_motor">
-            <mechanicalReduction>1</mechanicalReduction>
-        </actuator>
-    </transmission>
-    <transmission name="joint_2_trans">
-        <type>transmission_interface/SimpleTransmission</type>
-        <joint name="joint_2">
-            <hardwareInterface>hardware_interface/PositionJointInterface</hardwareInterface>
-        </joint>
-        <actuator name="joint_2_motor">
-            <mechanicalReduction>1</mechanicalReduction>
-        </actuator>
-    </transmission>
-    <transmission name="joint_3_trans">
-        <type>transmission_interface/SimpleTransmission</type>
-        <joint name="joint_3">
-            <hardwareInterface>hardware_interface/PositionJointInterface</hardwareInterface>
-        </joint>
-        <actuator name="joint_3_motor">
-            <mechanicalReduction>1</mechanicalReduction>
-        </actuator>
-    </transmission>
 </robot>

Commit message: fixed mimic behavior - working urdf model

File: install/eezybotarm_control/share/eezybotarm_control/description/eezybotarm.urdf.xacro (robot description, xacro)
@@ -34,5 +34,4 @@
         <axis xyz="0 0 -1"/>
         <limit effort="100" velocity="1.0" lower="-0.7854" upper="0.7854"/>
-        <!-- [-45,45] degrees -->
     </joint>
     <!-- LINK 1 -->
@@ -58,7 +57,5 @@
         <child link="link_2"/>
         <axis xyz="0 0 -1"/>
-        <!-- <limit effort="100" velocity="1.0" lower="-1.01229" upper="0.279253"/> -->
         <limit effort="100" velocity="1.0" lower="-0.279253" upper="1.01229"/>
-        <!-- [-35,55] degrees -->
     </joint>
     <!-- LINK 2 -->
@@ -78,12 +75,29 @@
         </collision>
     </link>
-    <!-- JOINT 3 (Elbow) -->
+    <!-- Intermediate Joint for Independent Movement (sharing rotation center with joint_2) -->
     <joint name="joint_3" type="revolute">
         <origin xyz="-0.021 0.133 -0.0105" rpy="0 0 0"/>
         <parent link="link_2"/>
+        <child link="link_2_5"/>
+        <axis xyz="0 0 -1"/>
+        <limit effort="100" velocity="1.0" lower="0" upper="1.22173"/>
+    </joint>
+    <!-- Intermediate Link -->
+    <link name="link_2_5">
+        <visual>
+            <origin xyz="0 0 0" rpy="0 0 0"/>
+            <geometry>
+                <sphere radius="0.001"/>
+            </geometry>
+        </visual>
+    </link>
+    <!-- JOINT 3 (Elbow) -->
+    <joint name="joint_2_5" type="revolute">
+        <origin xyz="0 0 0" rpy="0 0 0"/>
+        <parent link="link_2_5"/>
         <child link="link_3"/>
         <axis xyz="0 0 -1"/>
         <limit effort="100" velocity="1.0" lower="0" upper="1.22173"/>
-        <!-- [-70,20] degrees -->
+        <mimic joint="joint_2" multiplier="-1.0" offset="0"/>
     </joint>
     <!-- LINK 3 -->
